File: hardware/teensy-boom-jr/teensy-boom-jr.brd (EAGLE design)
At the start: 101.6 x 44.5 mm, 47 parts, among them U1 74AHC1G126, U2 74hc165, U3 74hc595

Commit message: Small updates to get ready to fab.
Parts:
- added FD1, FD2: FIDUCIALUFIDUCIAL, SparkFun-Aesthetics:MICRO-FIDUCIAL
- FRAME1: value FRAME-LETTERNO_PACKAGE -> FRAME-LETTER; device SparkFun-Aesthetics:DUMMY -> SparkFun-Aesthetics:CREATIVE_COMMONS
- J1: value (none) -> bypass buffer
- J2: value (none) -> To MCU
- J3: value (none) -> To Chain
- moved FRAME1 38.2 mm to (19.1, -7.62)
Other:
- board text added: "Byron Jacquot"
- board text added: "V01"
Changed lines of the file:
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@@
 <setting verticaltext="up"/>
 </settings>
-<grid distance="0.01" unitdist="inch" unit="inch" style="lines" multiple="1" display="yes" altdistance="0.001" altunitdist="inch" altunit="inch"/>
+<grid distance="0.05" unitdist="inch" unit="inch" style="lines" multiple="1" display="yes" altdistance="0.005" altunitdist="inch" altunit="inch"/>
 <layers>
 <layer number="1" name="Top" color="4" fill="1" visible="yes" active="yes"/>
@@
 <layer number="38" name="bTest" color="7" fill="1" visible="no" active="yes"/>
 <layer number="39" name="tKeepout" color="4" fill="11" visible="yes" active="yes"/>
-<layer number="40" name="bKeepout" color="1" fill="11" visible="no" active="yes"/>
+<layer number="40" name="bKeepout" color="1" fill="11" visible="yes" active="yes"/>
 <layer number="41" name="tRestrict" color="4" fill="10" visible="no" active="yes"/>
 <layer number="42" name="bRestrict" color="1" fill="10" visible="no" active="yes"/>
@@
 <layer number="49" name="Reference" color="7" fill="1" visible="no" active="yes"/>
 <layer number="50" name="dxf" color="7" fill="1" visible="no" active="no"/>
-<layer number="51" name="tDocu" color="6" fill="1" visible="no" active="yes"/>
+<layer number="51" name="tDocu" color="6" fill="1" visible="yes" active="yes"/>
 <layer number="52" name="bDocu" color="7" fill="1" visible="no" active="yes"/>
 <layer number="53" name="tGND_GNDA" color="7" fill="9" visible="no" active="no"/>
@@
 <board>
 <plain>
-<wire x1="0" y1="0" x2="101.6" y2="0" width="0" layer="20"/>
-<wire x1="101.6" y1="0" x2="101.6" y2="44.45" width="0" layer="20"/>
-<wire x1="101.6" y1="44.45" x2="0" y2="44.45" width="0" layer="20"/>
-<wire x1="0" y1="44.45" x2="0" y2="0" width="0" layer="20"/>
+<wire x1="0" y1="0" x2="101.6" y2="0" width="0.2032" layer="20"/>
+<wire x1="101.6" y1="0" x2="101.6" y2="44.45" width="0.2032" layer="20"/>
+<wire x1="101.6" y1="44.45" x2="0" y2="44.45" width="0.2032" layer="20"/>
+<wire x1="0" y1="44.45" x2="0" y2="0" width="0.2032" layer="20"/>
 <text x="6.35" y="6.35" size="3.81" layer="21" font="vector" ratio="15" align="top-center">1</text>
 <text x="19.05" y="6.35" size="3.81" layer="21" font="vector" ratio="15" align="top-center">2</text>
@@
 <text x="99.06" y="35.56" size="1.016" layer="22" font="vector" ratio="15" rot="MR0" align="center-left">LED</text>
 <text x="99.06" y="38.1" size="1.016" layer="22" font="vector" ratio="15" rot="MR0" align="center-left">BTN</text>
+<text x="7.62" y="1.27" size="1.778" layer="16" font="vector" ratio="15" rot="MR0">V01</text>
+<text x="49.53" y="-7.62" size="1.778" layer="51" font="vector">Byron Jacquot</text>
 </plain>
 <attributes>
@@
 </autorouter>
 <elements>
-<element name="FRAME1" library="SparkFun-Aesthetics" package="DUMMY" value="FRAME-LETTERNO_PACKAGE" x="-19.05" y="-10.16">
-<attribute name="DESIGNER" value="Nobody" x="-19.05" y="-10.16" size="1.778" layer="27" font="vector" ratio="15" display="off"/>
-<attribute name="VERSION" value="v01" x="-19.05" y="-10.16" size="1.778" layer="27" font="vector" ratio="15" display="off"/>
-</element>
 <element name="U3" library="teensy-synth" package="SO16" value="74hc595" x="31.75" y="36.83" rot="R270"/>
 <element name="D8" library="SparkFun-LED" package="LED3MM-NS" value="red" x="6.35" y="24.13" rot="R90"/>
@@
 <attribute name="PROD_ID" value="CAP-08604" x="38.1" y="36.83" size="1.778" layer="27" font="vector" ratio="15" rot="R90" display="off"/>
 </element>
-<element name="J3" library="SparkFun-Connectors" package="1X07_NO_SILK" value="" x="100.33" y="22.86" rot="R90"/>
+<element name="J3" library="SparkFun-Connectors" package="1X07_NO_SILK" value="To Chain" x="100.33" y="22.86" rot="R90"/>
 <element name="U2" library="teensy-synth" package="SO16" value="74hc165" x="69.85" y="36.83" rot="R270"/>
 <element name="C1" library="SparkFun-Capacitors" package="0603-CAP" value="0.1uF" x="76.2" y="36.83" rot="R90">
@@
 <attribute name="VALUE" value="74AHC1G126" x="12.446" y="36.576" size="1.778" layer="27" rot="R90" display="off"/>
 </element>
-<element name="J2" library="SparkFun-Connectors" package="1X07_NO_SILK" value="" x="1.27" y="22.86" rot="R90"/>
-<element name="J1" library="SparkFun-Connectors" package="1X02_NO_SILK" value="" x="13.716" y="40.386" rot="R180"/>
+<element name="J2" library="SparkFun-Connectors" package="1X07_NO_SILK" value="To MCU" x="1.27" y="22.86" rot="R90"/>
+<element name="J1" library="SparkFun-Connectors" package="1X02_NO_SILK" value="bypass buffer" x="13.716" y="40.386" rot="R180"/>
 <element name="H1" library="SparkFun-Electromechanical" package="STAND-OFF" value="STAND-OFF" x="6.35" y="40.64"/>
 <element name="H2" library="SparkFun-Electromechanical" package="STAND-OFF" value="STAND-OFF" x="12.7" y="3.81"/>
@@
 <element name="LOGO1" library="SparkFun-Aesthetics" package="OSHW-LOGO-S" value="OSHW-LOGOS" x="51.054" y="34.036"/>
 <element name="H5" library="SparkFun-Electromechanical" package="STAND-OFF" value="STAND-OFF" x="50.8" y="3.81"/>
+<element name="FRAME1" library="SparkFun-Aesthetics" package="CREATIVE_COMMONS" value="FRAME-LETTER" x="19.05" y="-7.62"/>
+<element name="FD1" library="SparkFun-Aesthetics" package="MICRO-FIDUCIAL" value="FIDUCIALUFIDUCIAL" x="2.54" y="3.81"/>
+<element name="FD2" library="SparkFun-Aesthetics" package="MICRO-FIDUCIAL" value="FIDUCIALUFIDUCIAL" x="87.63" y="43.18"/>
 </elements>
 <signals>
