File: hardware/teensy-boom-jr/teensy-boom-jr.sch (EAGLE design)
At the start: 47 parts, among them U1 74AHC1G126, U2 74hc165, U3 74hc595

Commit message: Small updates to get ready to fab.
Parts:
- added FD1, FD2: FIDUCIALUFIDUCIAL, SparkFun-Aesthetics:FIDUCIALUFIDUCIAL
- FRAME1: value FRAME-LETTERNO_PACKAGE -> FRAME-LETTER; device SparkFun-Aesthetics:FRAME-LETTERNO_PACKAGE -> SparkFun-Aesthetics:FRAME-LETTER
- J1: value (none) -> bypass buffer
- J2: value (none) -> To MCU
- J3: value (none) -> To Chain
Other:
- note added: "On board nearest host, install tri-state gate. On other boards in daisy-chain, simply strap J1."
- note removed: "On board nearest host, install tri-state gate. On other boards in daisy-chain, simply strap J3."
- moved on the sheet: C1, C2, D1, D2, D3, D4, D5, D6, D7, D8, J1, J2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
